File: Slaughter house.kicad_sch (KiCad schematic)
At the start: 7 parts, among them U1 DHT11

Commit message: Add files via upload
Connections:
- removed net +5V: DS1.2 (VDD), RV1.1, RV2.1, RV3.1, U1.1 (VDD)
- net Earth: no longer names the net of RV1.3
- removed net GND: BZ1.2 (-), DS1.1 (VSS), DS1.5 (R/W), RV2.3, RV3.3, U1.4 (GND)
- no-connect marks 25 -> 37
